File: LiIonUtilityBoard.kicad_pcb (KiCad board)
At the start: 2 copper layers, 0 parts

Commit message: Begin PCB Layout
Parts:
- added BT1: BATT, Connector_PinHeader_2.54mm:PinHeader_1x02_P2.54mm_Vertical, F.Cu at (123.3, 37.4)
- added C1: 2.2u, Capacitor_SMD:C_0603_1608Metric, F.Cu at (78.2, 44.4)
- added C10: 10u, Capacitor_SMD:C_0805_2012Metric, F.Cu at (74.0, 47.5)
- added C11: 10u, Capacitor_SMD:C_0805_2012Metric, F.Cu at (51.3, 63.3)
- added C12: 22u, Capacitor_SMD:C_0805_2012Metric, F.Cu at (82.0, 38.6)
- added C13: 22u, Capacitor_SMD:C_0805_2012Metric, F.Cu at (82.0, 41.6)
- added C14: 22u, Capacitor_SMD:C_0805_2012Metric, F.Cu at (69.0, 52.4)
- added C15: 0.47u, Capacitor_SMD:C_0402_1005Metric, F.Cu at (125.9, 55.7)
- added C2: 2.2u, Capacitor_SMD:C_0603_1608Metric, F.Cu at (64.7, 60.3)
- added C3: 2.2u, Capacitor_SMD:C_0603_1608Metric, F.Cu at (86.3, 38.3)
- added C4: 0.1u, Capacitor_SMD:C_0402_1005Metric, F.Cu at (75.5, 52.5)
- added C5: 0.1u, Capacitor_SMD:C_0402_1005Metric, F.Cu at (128.8, 40.4)
- added C6: 0.1u, Capacitor_SMD:C_0402_1005Metric, F.Cu at (128.4, 51.2)
- added C7: 10u, Capacitor_SMD:C_0805_2012Metric, F.Cu at (74.0, 44.5)
- added C8: 10u, Capacitor_SMD:C_0805_2012Metric, F.Cu at (63.4, 57.5)
- added C9: 10u, Capacitor_SMD:C_0805_2012Metric, F.Cu at (60.5, 60.5)
- added D1: INBOK, LED_SMD:LED_0603_1608Metric, F.Cu at (42.4, 63.2)
- added D2: STAT, LED_SMD:LED_0603_1608Metric, F.Cu at (46.4, 63.2)
- added J1: USB4510-03-1-A, LUBParts:GCT_USB4510-03-1-A_REVA, F.Cu at (155.8, 49.2)
- added J2: Conn_02x07_Odd_Even, Connector_PinHeader_2.54mm:PinHeader_2x07_P2.54mm_Vertical, F.Cu at (42.7, 39.4)
- added JP1: Jumper_3_Bridged12, Jumper:SolderJumper-3_P1.3mm_Open_Pad1.0x1.5mm_NumberLabels, F.Cu at (58.3, 56.0)
- added L1: 1u, Inductor_SMD:L_Taiyo-Yuden_NR-60xx, F.Cu at (51.5, 50.8)
- added L2: 1u, Inductor_SMD:L_Taiyo-Yuden_NR-60xx, F.Cu at (65.4, 40.9)
- added Q1: PMDPB30XN, LUBParts:DMN1025UFDB7, F.Cu at (121.1, 42.9)
- added R1: 10K, Resistor_SMD:R_0402_1005Metric, F.Cu at (85.7, 40.6)
- added R10: 100, Resistor_SMD:R_0402_1005Metric, F.Cu at (130.6, 39.9)
- added R11: 22, Resistor_SMD:R_0402_1005Metric, F.Cu at (131.8, 39.9)
- added R12: 10m, Resistor_SMD:R_0612_1632Metric, F.Cu at (120.4, 54.6)
- added R13: 10K, Resistor_SMD:R_0402_1005Metric, F.Cu at (64.2, 62.5)
- added R2: 10K, Resistor_SMD:R_0402_1005Metric, F.Cu at (77.7, 48.6)
- added R3: 10K, Resistor_SMD:R_0402_1005Metric, F.Cu at (68.2, 54.9)
- added R4: 10K, Resistor_SMD:R_0402_1005Metric, F.Cu at (54.9, 63.7)
- added R5: 1K, Resistor_SMD:R_0603_1608Metric, F.Cu at (67.6, 57.3)
- added R6: 1K, Resistor_SMD:R_0603_1608Metric, F.Cu at (60.3, 63.3)
- added R7: 1K, Resistor_SMD:R_0603_1608Metric, F.Cu at (130.1, 46.9)
- added R8: 18.2K, Resistor_SMD:R_0402_1005Metric, F.Cu at (81.7, 44.1)
- added R9: 2.26m, Resistor_SMD:R_2512_6332Metric, F.Cu at (125.8, 43.4)
- added TH1: THM, Connector_PinHeader_2.54mm:PinHeader_1x02_P2.54mm_Vertical, F.Cu at (57.8, 49.3)
- added U1: MAX77757JEFG420+, LUBParts:IC_MAX77757JEFG420+, F.Cu at (64.2, 53.5)
- added U2: bq298215, LUBParts:BQ298009RUGR, F.Cu at (130.1, 43.1)
- added U3: MAX17260SETD, Package_DFN_QFN:TDFN-14-1EP_3x3mm_P0.4mm_EP1.78x2.35mm, F.Cu at (125.8, 52.2)
- added U4: ISL91127IR, Package_DFN_QFN:QFN-20-1EP_4x4mm_P0.5mm_EP2.7x2.7mm_ThermalVias, F.Cu at (64.6, 47.8)
Routing:
- net Net-(C6-Pad1): track 0.00 -> 31.7 mm
- net Net-(Q1-Pad5): track 0.00 -> 17.0 mm, vias 0 -> 2
- net Net-(BT1-Pad1): track 0.00 -> 15.6 mm, vias 0 -> 2
- net Net-(Q1-Pad2): track 0.00 -> 14.5 mm, vias 0 -> 2
- net Net-(BT1-Pad2): track 0.00 -> 14.0 mm
- net GND: track 0.00 -> 6.48 mm, vias 0 -> 14
- net +BATT: track 0.00 -> 6.30 mm
- net Net-(C5-Pad1): track 0.00 -> 3.59 mm
- net Net-(Q1-Pad3): track 0.00 -> 2.95 mm
- net Net-(R11-Pad1): track 0.00 -> 2.62 mm
- net Net-(R7-Pad1): track 0.00 -> 2.29 mm
- net Net-(C15-Pad1): track 0.00 -> 1.55 mm
- added copper zone on B.Cu, net GND
- added copper zone on F.Cu, net GND
Other:
- board outline added: 40 x 75 mm

Commit message: Sync project status
Parts:
- removed BT1: BATT, Connector_PinHeader_2.54mm:PinHeader_1x02_P2.54mm_Vertical
- removed C1, C2, C3: 2.2u, Capacitor_SMD:C_0603_1608Metric
- removed C10, C11, C7, C8, C9: 10u, Capacitor_SMD:C_0805_2012Metric
- removed C12, C13, C14: 22u, Capacitor_SMD:C_0805_2012Metric
- removed C15: 0.47u, Capacitor_SMD:C_0402_1005Metric
- removed C4, C5, C6: 0.1u, Capacitor_SMD:C_0402_1005Metric
- removed D1: INBOK, LED_SMD:LED_0603_1608Metric
- removed D2: STAT, LED_SMD:LED_0603_1608Metric
- removed J1: USB4510-03-1-A, LUBParts:GCT_USB4510-03-1-A_REVA
- removed J2: Conn_02x07_Odd_Even, Connector_PinHeader_2.54mm:PinHeader_2x07_P2.54mm_Vertical
- removed JP1: Jumper_3_Bridged12, Jumper:SolderJumper-3_P1.3mm_Open_Pad1.0x1.5mm_NumberLabels
- removed L1, L2: 1u, Inductor_SMD:L_Taiyo-Yuden_NR-60xx
- removed Q1: PMDPB30XN, LUBParts:DMN1025UFDB7
- removed R1, R13, R2, R3, R4: 10K, Resistor_SMD:R_0402_1005Metric
- removed R10: 100, Resistor_SMD:R_0402_1005Metric
- removed R11: 22, Resistor_SMD:R_0402_1005Metric
- removed R12: 10m, Resistor_SMD:R_0612_1632Metric
- removed R5, R6, R7: 1K, Resistor_SMD:R_0603_1608Metric
- removed R8: 18.2K, Resistor_SMD:R_0402_1005Metric
- removed R9: 2.26m, Resistor_SMD:R_2512_6332Metric
- removed TH1: THM, Connector_PinHeader_2.54mm:PinHeader_1x02_P2.54mm_Vertical
- removed U1: MAX77757JEFG420+, LUBParts:IC_MAX77757JEFG420+
- removed U2: bq298215, LUBParts:BQ298009RUGR
- removed U3: MAX17260SETD, Package_DFN_QFN:TDFN-14-1EP_3x3mm_P0.4mm_EP1.78x2.35mm
- removed U4: ISL91127IR, Package_DFN_QFN:QFN-20-1EP_4x4mm_P0.5mm_EP2.7x2.7mm_ThermalVias
Routing:
- net Net-(C6-Pad1): track 31.7 -> 0.00 mm
- net Net-(Q1-Pad5): track 17.0 -> 0.00 mm, vias 2 -> 0
- net Net-(BT1-Pad1): track 15.6 -> 0.00 mm, vias 2 -> 0
- net Net-(Q1-Pad2): track 14.5 -> 0.00 mm, vias 2 -> 0
- net Net-(BT1-Pad2): track 14.0 -> 0.00 mm
- net GND: track 6.48 -> 0.00 mm, vias 14 -> 0
- net +BATT: track 6.30 -> 0.00 mm
- net Net-(C5-Pad1): track 3.59 -> 0.00 mm
- net Net-(Q1-Pad3): track 2.95 -> 0.00 mm
- net Net-(R11-Pad1): track 2.62 -> 0.00 mm
- net Net-(R7-Pad1): track 2.29 -> 0.00 mm
- net Net-(C15-Pad1): track 1.55 -> 0.00 mm
- removed copper zone on B.Cu, net GND
- removed copper zone on F.Cu, net GND
Other:
- board outline removed
