File: LiIonUtilityBoard.kicad_pcb (KiCad board)
At the start: 2 copper layers, 0 parts

Commit message: Finish Routing
Parts:
- added BT1: 12BHC186P-GR, LUBParts:12BHC186P-GR, B.Cu at (134.0, 66.0)
- added C1: 2.2u, Capacitor_SMD:C_0402_1005Metric, F.Cu at (110.5, 50.5)
- added C10: 22u, Capacitor_SMD:C_0805_2012Metric, F.Cu at (113.3, 50.5)
- added C11: 47u, Capacitor_SMD:CP_Elec_5x5.3, F.Cu at (169.0, 66.0)
- added C2: 2.2u, Capacitor_SMD:C_0402_1005Metric, F.Cu at (114.3, 60.5)
- added C3: 2.2u, Capacitor_SMD:C_0402_1005Metric, F.Cu at (120.6, 54.1)
- added C4: 10u, Capacitor_SMD:C_0603_1608Metric, F.Cu at (116.6, 57.9)
- added C5: 10u, Capacitor_SMD:C_0603_1608Metric, F.Cu at (113.3, 48.5)
- added C6: 10u, Capacitor_SMD:C_0603_1608Metric, F.Cu at (116.6, 54.9)
- added C7: 10u, Capacitor_SMD:C_0603_1608Metric, F.Cu at (118.3, 54.9)
- added C8: 0.1u, Capacitor_SMD:C_0402_1005Metric, F.Cu at (160.3, 73.9)
- added C9: 0.1u, Capacitor_SMD:C_0402_1005Metric, F.Cu at (110.0, 53.3)
- added D1: INBOK, LED_SMD:LED_0603_1608Metric, F.Cu at (102.4, 48.0)
- added D2: STAT, LED_SMD:LED_0603_1608Metric, F.Cu at (102.4, 50.0)
- added J1: USBC_Swapped, Connector_USB:USB_C_Receptacle_GCT_USB4085, F.Cu at (92.0, 63.0)
- added J2: Output, LUBParts:CUI_TB002-500-03BE, F.Cu at (177.3, 61.0)
- added JP1: IFAST1, Jumper:SolderJumper-2_P1.3mm_Bridged_Pad1.0x1.5mm, F.Cu at (119.4, 80.3)
- added JP2: IFAST2, Jumper:SolderJumper-2_P1.3mm_Bridged_Pad1.0x1.5mm, F.Cu at (124.5, 80.3)
- added JP3: THM_EN, Jumper:SolderJumper-3_P1.3mm_Bridged12_Pad1.0x1.5mm_NumberLabels, F.Cu at (107.4, 80.3)
- added L1: 0.47u, Inductor_SMD:L_1008_2520Metric, F.Cu at (118.1, 51.7)
- added Q1: PMDPB30XN, LUBParts:SON65P200X200X65-8N, F.Cu at (114.9, 66.0)
- added R1: 10K, Resistor_SMD:R_0402_1005Metric, F.Cu at (114.3, 61.7)
- added R10: 9.0m, Resistor_SMD:R_0603_1608Metric, F.Cu at (162.8, 75.7)
- added R11: 100, Resistor_SMD:R_0402_1005Metric, F.Cu at (160.3, 71.6)
- added R12: 22, Resistor_SMD:R_0402_1005Metric, F.Cu at (162.1, 70.1)
- added R2: 10K, Resistor_SMD:R_0402_1005Metric, F.Cu at (111.5, 80.3)
- added R3: 10K, Resistor_SMD:R_0402_1005Metric, F.Cu at (114.3, 58.9)
- added R4: 1K, Resistor_SMD:R_0402_1005Metric, F.Cu at (107.7, 53.6)
- added R5: 1K, Resistor_SMD:R_0402_1005Metric, F.Cu at (107.7, 54.9)
- added R6: 1K, Resistor_SMD:R_0402_1005Metric, F.Cu at (157.5, 72.6)
- added R7: 6.65K, Resistor_SMD:R_0402_1005Metric, F.Cu at (114.6, 76.2)
- added R8: 7.32K, Resistor_SMD:R_0402_1005Metric, F.Cu at (119.4, 78.0)
- added R9: 8.66K, Resistor_SMD:R_0402_1005Metric, F.Cu at (124.5, 78.0)
- added TH1: THM, Connector_PinHeader_2.54mm:PinHeader_1x02_P2.54mm_Vertical, F.Cu at (93.5, 82.3)
- added U1: MAX77757JEFG420+, LUBParts:IC_MAX77757JEFG420+, F.Cu at (112.7, 55.6)
- added U2: bq298019, LUBParts:BQ298009RUGR, F.Cu at (163.1, 72.8)
Routing:
- net Net-(BT1-Pad1): track 0.00 -> 89.5 mm
- net +SYS: track 0.00 -> 86.9 mm
- net /ENBST: track 0.00 -> 73.2 mm, vias 0 -> 2
- net +BATT: track 0.00 -> 59.4 mm, vias 0 -> 2
- net Net-(Q1-Pad2): track 0.00 -> 54.9 mm, vias 0 -> 2
- net Net-(Q1-Pad5): track 0.00 -> 51.4 mm, vias 0 -> 2
- net Net-(J1-PadB5): track 0.00 -> 37.8 mm, vias 0 -> 2
- net Net-(C1-Pad2): track 0.00 -> 36.8 mm
- net Net-(BT1-Pad2): track 0.00 -> 35.6 mm
- net Net-(JP3-Pad2): track 0.00 -> 26.0 mm, vias 0 -> 2
- net Net-(J1-PadA7): track 0.00 -> 25.5 mm
- net Net-(J1-PadA6): track 0.00 -> 24.7 mm
- net Net-(J1-PadA5): track 0.00 -> 22.7 mm
- net /IFAST: track 0.00 -> 19.0 mm, vias 0 -> 2
- net GND: track 0.00 -> 17.8 mm, vias 0 -> 30
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- added copper zone on F.Cu, net +SYS
- added copper zone on B.Cu, net GND
- added copper zone on F.Cu, net GND
Other:
- board outline added: 96 x 40 mm
