File: LiIonUtilityBoard.kicad_pcb (KiCad board)
At the start: 2 copper layers, 96 x 40 mm, 36 parts, among them J1 USBC_Swapped, J2 Output, Q1 PMDPB30XN, U1 MAX77757JEFG420+, U2 bq298019

Commit message: Final Rev 0.1 PCB
Parts:
- TH1: moved to B.Cu
- moved C11 0.80 mm to (168.2, 66.0)
- turned TH1 to 0 degrees
Routing:
- net Net-(JP3-Pad2): track 26.0 -> 32.2 mm
- net GND: track 17.8 -> 11.8 mm, vias 30 -> 258
- net /IFAST: track 19.0 -> 21.4 mm
- net Net-(C1-Pad2): track 36.8 -> 35.6 mm
- net Net-(C9-Pad1): track 13.6 -> 14.3 mm
Other:
- board text added: "(Flashing - Charging, On - Done)"
- board text added: "1: SYS Out 2: GND 3: Boost Enable"
- board text added: "Charge Status"
- board text added: "Input Good"
- board text added: "Jumper Configuration: JP 1 and 2 Closed: 1A JP 2 Closed: 2A All Open: 3A JP3 1-2 Closed: Enable Thermistor JP3 2-3 Closed: Disable Thermistor"
- board text added: "LiIon Utility Board (Integrated Batteries) Version 0.1 © 2023 Sam Bach"
- board text added: "Thermistor Input"
